Commit message: refactor():更改gripper关节名，由joint*更改为gripper_joint*

File: piper/urdf/piper_description.urdf (robot description, URDF)
Before this commit: robot piper, 10 links, 9 joints
Joints:
- removed joint joint7
- removed joint joint8
- added joint gripper_joint1: type prismatic, parent gripper_base, child link7, origin xyz=0 0 0.1358 rpy=1.5708 0 0, axis 0 0 1, limit lower=0 upper=0.035 effort=10 velocity=1
- added joint gripper_joint2: type prismatic, parent gripper_base, child link8, origin xyz=0 0 0.1358 rpy=1.5708 0 -3.1416, axis 0 0 -1, limit lower=-0.035 upper=0 effort=10 velocity=1

File: piper/urdf/piper_description.xacro (robot description, xacro)
@@ -429,5 +429,5 @@
   </link>
   <joint
-    name="joint7"
+    name="gripper_joint1"
     type="prismatic">
     <origin
@@ -487,5 +487,5 @@
   </link>
   <joint
-    name="joint8"
+    name="gripper_joint2"
     type="prismatic">
     <origin
@@ -523,6 +523,6 @@
   <xacro:transmission_block tran_name="tran5" joint_name="joint5" motor_name="motor5"/>
   <xacro:transmission_block tran_name="tran6" joint_name="joint6" motor_name="motor6"/>
-  <xacro:transmission_block tran_name="tran7" joint_name="joint7" motor_name="motor7"/>
-  <xacro:transmission_block tran_name="tran8" joint_name="joint8" motor_name="motor8"/>
+  <xacro:transmission_block tran_name="tran7" joint_name="gripper_joint1" motor_name="motor7"/>
+  <xacro:transmission_block tran_name="tran8" joint_name="gripper_joint2" motor_name="motor8"/>
 <!-- gazebo -->
   <gazebo>

File: piper/urdf/piper_description_gazebo.xacro (robot description, xacro)
@@ -429,5 +429,5 @@
   </link>
   <joint
-    name="joint7"
+    name="gripper_joint1"
     type="prismatic">
     <origin
@@ -487,5 +487,5 @@
   </link>
   <joint
-    name="joint8"
+    name="gripper_joint2"
     type="prismatic">
     <origin
@@ -599,15 +599,15 @@
           <state_interface name="velocity"/>
       </joint>
-      <joint name="joint7">
-          <command_interface name="position">
-              <param name="min">-1</param>
-              <param name="max">1</param>
-          </command_interface>
-          <state_interface name="position">
-              <param name="initial_value">0.0</param>
-          </state_interface>
-          <state_interface name="velocity"/>
-      </joint>
-      <joint name="joint8">
+      <joint name="gripper_joint1">
+          <command_interface name="position">
+              <param name="min">-1</param>
+              <param name="max">1</param>
+          </command_interface>
+          <state_interface name="position">
+              <param name="initial_value">0.0</param>
+          </state_interface>
+          <state_interface name="velocity"/>
+      </joint>
+      <joint name="gripper_joint2">
           <command_interface name="position">
               <param name="min">-1</param>

File: piper/urdf/piper_description_old.urdf (robot description, URDF)
Before this commit: robot piper, 10 links, 9 joints
Joints:
- removed joint joint7
- removed joint joint8
- added joint gripper_joint1: type prismatic, parent gripper_base, child link7, origin xyz=0 0 0.1358 rpy=1.5708 0 0, axis 0 0 1, limit lower=0 upper=0.035 effort=10 velocity=1
- added joint gripper_joint2: type prismatic, parent gripper_base, child link8, origin xyz=0 0 0.1358 rpy=1.5708 0 -3.1416, axis 0 0 -1, limit lower=-0.035 upper=0 effort=10 velocity=1

File: piper/urdf/piper_description_v100_camera.urdf (robot description, URDF)
Before this commit: robot piper_camera, 10 links, 9 joints
Joints:
- removed joint joint7
- removed joint joint8
- added joint gripper_joint1: type prismatic, parent link6, child link7, origin xyz=0 0 0.13503 rpy=1.5708 0 1.5708, axis 0 0 -1, limit lower=0 upper=0.05 effort=100 velocity=1
- added joint gripper_joint2: type prismatic, parent link6, child link8, origin xyz=0 0 0.13503 rpy=-1.5708 0 1.5708, axis 0 0 1, limit lower=-0.05 upper=0 effort=100 velocity=1

File: piper/urdf/piper_description_v100_realsense_camera.urdf (robot description, URDF)
Before this commit: robot piper_camera, 10 links, 10 joints
Joints:
- removed joint joint7
- removed joint joint8
- added joint gripper_joint1: type prismatic, parent link6, child link7, origin xyz=0 0 0.13503 rpy=1.5708 0 1.5708, axis 0 0 -1, limit lower=0 upper=0.05 effort=100 velocity=1
- added joint gripper_joint2: type prismatic, parent link6, child link8, origin xyz=0 0 0.13503 rpy=-1.5708 0 1.5708, axis 0 0 1, limit lower=-0.05 upper=0 effort=100 velocity=1

File: piper/urdf/piper_description_v100_realsense_camera_v2.urdf (robot description, URDF)
Before this commit: robot piper_camera, 13 links, 12 joints
Joints:
- removed joint joint7
- removed joint joint8
- added joint gripper_joint1: type prismatic, parent link6, child link7, origin xyz=0 0 0.13503 rpy=1.5708 0 1.5708, axis 0 0 -1, limit lower=0 upper=0.05 effort=100 velocity=1
- added joint gripper_joint2: type prismatic, parent link6, child link8, origin xyz=0 0 0.13503 rpy=-1.5708 0 1.5708, axis 0 0 1, limit lower=-0.05 upper=0 effort=100 velocity=1

File: piper/urdf/piper_description_v100_realsense_camera_v2_dark.urdf (robot description, URDF)
Before this commit: robot piper_camera, 13 links, 12 joints
Joints:
- removed joint joint7
- removed joint joint8
- added joint gripper_joint1: type prismatic, parent link6, child link7, origin xyz=0 0 0.13503 rpy=1.5708 0 1.5708, axis 0 0 -1, limit lower=0 upper=0.05 effort=100 velocity=1
- added joint gripper_joint2: type prismatic, parent link6, child link8, origin xyz=0 0 0.13503 rpy=-1.5708 0 1.5708, axis 0 0 1, limit lower=-0.05 upper=0 effort=100 velocity=1

File: piper_h/urdf/piper_h_description.xacro (robot description, xacro)
@@ -368,5 +368,5 @@
   </collision>
 </link>
-    <joint name="joint7" type="prismatic">
+    <joint name="gripper_joint1" type="prismatic">
         <origin xyz="0 0 0.13503" rpy="1.5708 0 0" />
         <parent link="link6" />
@@ -405,5 +405,5 @@
         </collision>
     </link>
-    <joint name="joint8" type="prismatic">
+    <joint name="gripper_joint2" type="prismatic">
         <origin xyz="0 0 0.13503" rpy="-1.5708 0 0" />
         <parent link="link6" />

File: piper_h/urdf/piper_h_description_d435.urdf (robot description, URDF)
Before this commit: robot piper_l_camera, 13 links, 12 joints
Joints:
- removed joint joint7
- removed joint joint8
- added joint gripper_joint1: type prismatic, parent link6, child link7, origin xyz=0 0 0.13503 rpy=1.5708 0 0, axis 0 0 -1, limit lower=0 upper=0.05 effort=100 velocity=1
- added joint gripper_joint2: type prismatic, parent link6, child link8, origin xyz=0 0 0.13503 rpy=-1.5708 0 0, axis 0 0 1, limit lower=-0.05 upper=0 effort=100 velocity=1

File: piper_h/urdf/piper_h_description_d435_dark.urdf (robot description, URDF)
Before this commit: robot piper_l_camera, 13 links, 12 joints
Joints:
- removed joint joint7
- removed joint joint8
- added joint gripper_joint1: type prismatic, parent link6, child link7, origin xyz=0 0 0.13503 rpy=1.5708 0 0, axis 0 0 -1, limit lower=0 upper=0.05 effort=100 velocity=1
- added joint gripper_joint2: type prismatic, parent link6, child link8, origin xyz=0 0 0.13503 rpy=-1.5708 0 0, axis 0 0 1, limit lower=-0.05 upper=0 effort=100 velocity=1

File: piper_l/urdf/piper_l_description.xacro (robot description, xacro)
@@ -379,5 +379,5 @@
   </collision>
 </link>
-    <joint name="joint7" type="prismatic">
+    <joint name="gripper_joint1r_joint_1" type="prismatic">
         <origin xyz="0 0 0.13503" rpy="1.5708 0 0" />
         <parent link="link6" />
@@ -416,5 +416,5 @@
         </collision>
     </link>
-    <joint name="joint8" type="prismatic">
+    <joint name="gripper_joint2" type="prismatic">
         <origin xyz="0 0 0.13503" rpy="-1.5708 0 0" />
         <parent link="link6" />

File: piper_l/urdf/piper_l_description_d435.urdf (robot description, URDF)
Before this commit: robot piper_l_camera, 13 links, 12 joints
Joints:
- removed joint joint7
- removed joint joint8
- added joint gripper_joint1r_joint_1: type prismatic, parent link6, child link7, origin xyz=0 0 0.13503 rpy=1.5708 0 0, axis 0 0 -1, limit lower=0 upper=0.05 effort=100 velocity=1
- added joint gripper_joint2: type prismatic, parent link6, child link8, origin xyz=0 0 0.13503 rpy=-1.5708 0 0, axis 0 0 1, limit lower=-0.05 upper=0 effort=100 velocity=1

File: piper_l/urdf/piper_l_description_d435_dark.urdf (robot description, URDF)
Before this commit: robot piper_l_camera, 13 links, 12 joints
Joints:
- removed joint joint7
- removed joint joint8
- added joint gripper_joint1: type prismatic, parent link6, child link7, origin xyz=0 0 0.13503 rpy=1.5708 0 0, axis 0 0 -1, limit lower=0 upper=0.05 effort=100 velocity=1
- added joint gripper_joint2: type prismatic, parent link6, child link8, origin xyz=0 0 0.13503 rpy=-1.5708 0 0, axis 0 0 1, limit lower=-0.05 upper=0 effort=100 velocity=1

File: piper_x/urdf/piper_x_description copy.urdf (robot description, URDF)
Before this commit: robot piper_x_description, 9 links, 8 joints
Joints:
- removed joint joint7
- removed joint joint8
- added joint gripper_joint1: type prismatic, parent link6, child link7, origin xyz=0 0 0.13503 rpy=1.5708 0 1.5708, axis 0 0 -1, limit lower=0 upper=0.05 effort=100 velocity=1
- added joint gripper_joint2: type prismatic, parent link6, child link8, origin xyz=0 0 0.13503 rpy=-1.5708 0 1.5708, axis 0 0 1, limit lower=-0.05 upper=0 effort=100 velocity=1

File: piper_x/urdf/piper_x_description.urdf (robot description, URDF)
Before this commit: robot piper_x_description, 10 links, 9 joints
Joints:
- removed joint joint7
- removed joint joint8
- added joint gripper_joint1: type prismatic, parent gripper_base, child link7, origin xyz=0 0 0.13503 rpy=1.5708 0 1.5708, axis 0 0 -1, limit lower=0 upper=0.05 effort=100 velocity=1
- added joint gripper_joint2: type prismatic, parent gripper_base, child link8, origin xyz=0 0 0.13503 rpy=-1.5708 0 1.5708, axis 0 0 1, limit lower=-0.05 upper=0 effort=100 velocity=1

File: piper_x/urdf/piper_x_description.xacro (robot description, xacro)
@@ -444,5 +444,5 @@
     </collision>
   </link>
-    <joint name="joint7" type="prismatic">
+    <joint name="gripper_joint1" type="prismatic">
         <origin xyz="0 0 0.13503" rpy="1.5708 0 1.5708" />
         <parent link="gripper_base" />
@@ -481,5 +481,5 @@
         </collision>
     </link>
-    <joint name="joint8" type="prismatic">
+    <joint name="gripper_joint2" type="prismatic">
         <origin xyz="0 0 0.13503" rpy="-1.5708 0 1.5708" />
         <parent link="gripper_base" />

File: piper_x/urdf/piper_x_description_d435.urdf (robot description, URDF)
Before this commit: robot piper_x_camera, 14 links, 13 joints
Joints:
- removed joint joint7
- removed joint joint8
- added joint gripper_joint1: type prismatic, parent gripper_base, child link7, origin xyz=0 0 0.13503 rpy=1.5708 0 1.5708, axis 0 0 -1, limit lower=0 upper=0.05 effort=100 velocity=1
- added joint gripper_joint2: type prismatic, parent gripper_base, child link8, origin xyz=0 0 0.13503 rpy=-1.5708 0 1.5708, axis 0 0 1, limit lower=-0.05 upper=0 effort=100 velocity=1

File: piper_x/urdf/piper_x_description_d435_dark.urdf (robot description, URDF)
Before this commit: robot piper_x_camera, 14 links, 13 joints
Joints:
- removed joint joint7
- removed joint joint8
- added joint gripper_joint1: type prismatic, parent gripper_base, child link7, origin xyz=0 0 0.13503 rpy=1.5708 0 1.5708, axis 0 0 -1, limit lower=0 upper=0.05 effort=100 velocity=1
- added joint gripper_joint2: type prismatic, parent gripper_base, child link8, origin xyz=0 0 0.13503 rpy=-1.5708 0 1.5708, axis 0 0 1, limit lower=-0.05 upper=0 effort=100 velocity=1
